Commit message: Updated xacro file for parts (added base_link)

File: motor_description/urdf/robot_parts_move.xacro (robot description, xacro)
@@ -1,10 +1,31 @@
 <?xml version="1.0"?>
 <robot name="steerable_wheel_robot" xmlns:xacro="http://www.ros.org/wiki/xacro">
-  <!-- World link -->
-  <link name="world"/>
-  <!-- Vertical cylinder link -->
-  <link name="cylinder_link">
+  <!-- Base link (cube) -->
+  <link name="base_link">
     <visual>
-      <origin xyz="0 0 0.5" rpy="0 0 0"/>
+      <origin xyz="0 0 1.15" rpy="0 0 0"/>
+      <geometry>
+        <box size="0.4 0.4 0.2"/>
+      </geometry>
+      <material name="blue">
+        <color rgba="0 0 1 1"/>
+      </material>
+    </visual>
+    <collision>
+      <origin xyz="0 0 1.15" rpy="0 0 0"/>
+      <geometry>
+        <box size="0.4 0.4 0.2"/>
+      </geometry>
+    </collision>
+    <inertial>
+      <mass value="2.0"/>
+      <origin xyz="0 0 1.15" rpy="0 0 0"/>
+      <inertia ixx="0.1" iyy="0.1" izz="0.1" ixy="0" ixz="0" iyz="0"/>
+    </inertial>
+  </link>
+  <!-- Shaft (vertical cylinder) -->
+  <link name="shaft">
+    <visual>
+      <origin xyz="0 0 0.65" rpy="0 0 0"/>
       <geometry>
         <cylinder radius="0.05" length="1.0"/>
@@ -15,5 +36,5 @@
     </visual>
     <collision>
-      <origin xyz="0 0 0.5" rpy="0 0 0"/>
+      <origin xyz="0 0 0.65" rpy="0 0 0"/>
       <geometry>
         <cylinder radius="0.05" length="1.0"/>
@@ -22,14 +43,14 @@
     <inertial>
       <mass value="1.0"/>
-      <origin xyz="0 0 0.5" rpy="0 0 0"/>
-      <inertia ixx="0.0834375" ixy="0" ixz="0" iyy="0.0834375" iyz="0" izz="0.00125"/>
+      <origin xyz="0 0 0.65" rpy="0 0 0"/>
+      <inertia ixx="0.05" iyy="0.05" izz="0.001" ixy="0" ixz="0" iyz="0"/>
     </inertial>
   </link>
-  <!-- Wheel link (cylinder for traction) -->
-  <link name="wheel_link">
+  <!-- Wheel (horizontal cylinder) -->
+  <link name="wheel">
     <visual>
       <origin xyz="0 0 0" rpy="1.5708 0 0"/>
       <geometry>
-        <cylinder radius="0.1" length="0.05"/>
+        <cylinder radius="0.15" length="0.08"/>
       </geometry>
       <material name="black">
@@ -40,28 +61,26 @@
       <origin xyz="0 0 0" rpy="1.5708 0 0"/>
       <geometry>
-        <cylinder radius="0.1" length="0.05"/>
+        <cylinder radius="0.15" length="0.08"/>
       </geometry>
     </collision>
     <inertial>
-      <mass value="0.2"/>
-      <inertia ixx="0.0002667" ixy="0" ixz="0" iyy="0.0002667" iyz="0" izz="0.0002"/>
+      <mass value="0.5"/>
+      <inertia ixx="0.001" iyy="0.001" izz="0.0008" ixy="0" ixz="0" iyz="0"/>
     </inertial>
   </link>
-  <!-- Revolute joint for steering (-90 to 90 degrees) -->
+  <!-- Revolute joint: base_link ↔ shaft (steering) -->
   <joint name="steer_joint" type="revolute">
-    <parent link="world"/>
-    <child link="cylinder_link"/>
+    <parent link="base_link"/>
+    <child link="shaft"/>
     <origin xyz="0 0 0" rpy="0 0 0"/>
     <axis xyz="0 0 1"/>
     <limit lower="-1.5708" upper="1.5708" velocity="1.0" effort="50"/>
-    <dynamics damping="0.05" friction="0.05"/>
   </joint>
-  <!-- Continuous joint for wheel traction -->
+  <!-- Continuous joint: shaft ↔ wheel (traction) -->
   <joint name="trac_joint" type="continuous">
-    <parent link="cylinder_link"/>
-    <child link="wheel_link"/>
-    <origin xyz="0 0 1.0" rpy="0 0 0"/>
+    <parent link="shaft"/>
+    <child link="wheel"/>
+    <origin xyz="0 0 0.15" rpy="0 0 0"/>
     <axis xyz="0 1 0"/>
-    <dynamics damping="0.01" friction="0.01"/>
   </joint>
 </robot>

Commit message: Removed inertia from base_link (since it's root link)

File: motor_description/urdf/robot_parts_move.xacro (robot description, xacro)
@@ -18,9 +18,4 @@
       </geometry>
     </collision>
-    <inertial>
-      <mass value="2.0"/>
-      <origin xyz="0 0 1.15" rpy="0 0 0"/>
-      <inertia ixx="0.1" iyy="0.1" izz="0.1" ixy="0" ixz="0" iyz="0"/>
-    </inertial>
   </link>
   <!-- Shaft (vertical cylinder) -->

Commit message: Added lidar link to the urdf file

File: motor_description/urdf/robot_parts_move.xacro (robot description, xacro)
@@ -16,4 +16,22 @@
       <geometry>
         <box size="0.4 0.4 0.2"/>
+      </geometry>
+    </collision>
+  </link>
+  <!-- LiDAR link -->
+  <link name="lidar_nav_link">
+    <visual>
+      <origin xyz="0.037 0 0.9" rpy="0 0 0"/>
+      <geometry>
+        <cylinder radius="0.1" length="0.04"/>
+      </geometry>
+      <material name="blue">
+        <color rgba="0 0 1 1"/>
+      </material>
+    </visual>
+    <collision>
+      <origin xyz="0.037 0 0.9" rpy="0 0 0"/>
+      <geometry>
+        <cylinder radius="0.1" length="0.04"/>
       </geometry>
     </collision>
@@ -64,4 +82,10 @@
     </inertial>
   </link>
+  <!-- Fixed joint: base_link ↔ lidar -->
+  <joint name="lidar_joint" type="fixed">
+    <parent link="base_link"/>
+    <child link="lidar_nav_link"/>
+    <origin xyz="0 0 0" rpy="0 0 0"/>
+  </joint>
   <!-- Revolute joint: base_link ↔ shaft (steering) -->
   <joint name="steer_joint" type="revolute">

Commit message: Updated URDF file

File: motor_description/urdf/robot_parts_move.xacro (robot description, xacro)
@@ -86,5 +86,5 @@
     <parent link="base_link"/>
     <child link="lidar_nav_link"/>
-    <origin xyz="0 0 0" rpy="0 0 0"/>
+    <origin xyz="0 0 0" rpy="0 0 3.1416"/>
   </joint>
   <!-- Revolute joint: base_link ↔ shaft (steering) -->

Commit message: Updated URDF file

File: motor_description/urdf/robot_parts_move.xacro (robot description, xacro)
@@ -65,5 +65,5 @@
       <origin xyz="0 0 0" rpy="1.5708 0 0"/>
       <geometry>
-        <cylinder radius="0.15" length="0.08"/>
+        <cylinder radius="0.124" length="0.08"/>
       </geometry>
       <material name="black">
@@ -74,5 +74,5 @@
       <origin xyz="0 0 0" rpy="1.5708 0 0"/>
       <geometry>
-        <cylinder radius="0.15" length="0.08"/>
+        <cylinder radius="0.124" length="0.08"/>
       </geometry>
     </collision>
@@ -86,5 +86,5 @@
     <parent link="base_link"/>
     <child link="lidar_nav_link"/>
-    <origin xyz="0 0 0" rpy="0 0 3.1416"/>
+    <origin xyz="0 0 0.874" rpy="0 0 3.1416"/>
   </joint>
   <!-- Revolute joint: base_link ↔ shaft (steering) -->
@@ -92,5 +92,5 @@
     <parent link="base_link"/>
     <child link="shaft"/>
-    <origin xyz="0 0 0" rpy="0 0 0"/>
+    <origin xyz="0 0 0.154" rpy="0 0 0"/>
     <axis xyz="0 0 1"/>
     <limit lower="-1.5708" upper="1.5708" velocity="1.0" effort="50"/>
@@ -100,5 +100,5 @@
     <parent link="shaft"/>
     <child link="wheel"/>
-    <origin xyz="0 0 0.15" rpy="0 0 0"/>
+    <origin xyz="0 0 -0.03" rpy="0 0 0"/>
     <axis xyz="0 1 0"/>
   </joint>

Commit message: Updated URDF file

File: motor_description/urdf/robot_parts_move.xacro (robot description, xacro)
@@ -86,5 +86,5 @@
     <parent link="base_link"/>
     <child link="lidar_nav_link"/>
-    <origin xyz="0 0 0.874" rpy="0 0 3.1416"/>
+    <origin xyz="0.037 0 0.874" rpy="0 0 3.1416"/>
   </joint>
   <!-- Revolute joint: base_link ↔ shaft (steering) -->

Commit message: Updated URDF file

File: motor_description/urdf/robot_parts_move.xacro (robot description, xacro)
@@ -100,5 +100,5 @@
     <parent link="shaft"/>
     <child link="wheel"/>
-    <origin xyz="0 0 -0.03" rpy="0 0 0"/>
+    <origin xyz="0 -0.0055 -0.03" rpy="0 0 0"/>
     <axis xyz="0 1 0"/>
   </joint>

Commit message: Updated URDF file

File: motor_description/urdf/robot_parts_move.xacro (robot description, xacro)
@@ -86,5 +86,5 @@
     <parent link="base_link"/>
     <child link="lidar_nav_link"/>
-    <origin xyz="0.037 0 0.874" rpy="0 0 3.1416"/>
+    <origin xyz="0.37 0 0.874" rpy="0 0 3.1416"/>
   </joint>
   <!-- Revolute joint: base_link ↔ shaft (steering) -->

Commit message: Updated URDF file

File: motor_description/urdf/robot_parts_move.xacro (robot description, xacro)
@@ -86,5 +86,5 @@
     <parent link="base_link"/>
     <child link="lidar_nav_link"/>
-    <origin xyz="0.37 0 0.874" rpy="0 0 3.1416"/>
+    <origin xyz="0.037 0 0.874" rpy="0 0 3.1416"/>
   </joint>
   <!-- Revolute joint: base_link ↔ shaft (steering) -->
@@ -92,7 +92,7 @@
     <parent link="base_link"/>
     <child link="shaft"/>
-    <origin xyz="0 0 0.154" rpy="0 0 0"/>
+    <origin xyz="0 -0.0055 0.154" rpy="0 0 0"/>
     <axis xyz="0 0 1"/>
-    <limit lower="-1.5708" upper="1.5708" velocity="1.0" effort="50"/>
+    <limit lower="-1.5708" upper="1.5708" velocity="1.4" effort="200"/>
   </joint>
   <!-- Continuous joint: shaft ↔ wheel (traction) -->
@@ -100,5 +100,5 @@
     <parent link="shaft"/>
     <child link="wheel"/>
-    <origin xyz="0 -0.0055 -0.03" rpy="0 0 0"/>
+    <origin xyz="0 0 -0.03" rpy="0 0 0"/>
     <axis xyz="0 1 0"/>
   </joint>

Commit message: Updated URDF file (test)

File: motor_description/urdf/robot_parts_move.xacro (robot description, xacro)
@@ -86,5 +86,5 @@
     <parent link="base_link"/>
     <child link="lidar_nav_link"/>
-    <origin xyz="0.037 0 0.874" rpy="0 0 3.1416"/>
+    <origin xyz="1.027 0 0.874" rpy="0 0 3.1416"/>
   </joint>
   <!-- Revolute joint: base_link ↔ shaft (steering) -->
@@ -92,5 +92,5 @@
     <parent link="base_link"/>
     <child link="shaft"/>
-    <origin xyz="0 -0.0055 0.154" rpy="0 0 0"/>
+    <origin xyz="0.99 -0.0055 0.154" rpy="0 0 0"/>
     <axis xyz="0 0 1"/>
     <limit lower="-1.5708" upper="1.5708" velocity="1.4" effort="200"/>

Commit message: Updated lidar height (for the local cost map issue)

File: motor_description/urdf/robot_parts_move.xacro (robot description, xacro)
@@ -86,5 +86,5 @@
     <parent link="base_link"/>
     <child link="lidar_nav_link"/>
-    <origin xyz="1.027 0 0.874" rpy="0 0 3.1416"/>
+    <origin xyz="1.027 0 0.779" rpy="0 0 3.1416"/> <!-- z = 0.874 -->
   </joint>
   <!-- Revolute joint: base_link ↔ shaft (steering) -->

Commit message: Changed lidar (to sick)

File: motor_description/urdf/robot_parts_move.xacro (robot description, xacro)
@@ -86,5 +86,6 @@
     <parent link="base_link"/>
     <child link="lidar_nav_link"/>
-    <origin xyz="1.027 0 0.779" rpy="0 0 3.1416"/> <!-- z = 0.874 -->
+    <!-- <origin xyz="1.027 0 0.779" rpy="0 0 3.1416"/> z = 0.874 -->
+    <origin xyz="1.027 0 0.779" rpy="0 0 3.1416"/>
   </joint>
   <!-- Revolute joint: base_link ↔ shaft (steering) -->

Commit message: Brought back the navigation lidar (pf lidar)

File: motor_description/urdf/robot_parts_move.xacro (robot description, xacro)
@@ -86,6 +86,6 @@
     <parent link="base_link"/>
     <child link="lidar_nav_link"/>
-    <!-- <origin xyz="1.027 0 0.779" rpy="0 0 3.1416"/> z = 0.874 -->
-    <origin xyz="1.027 0 0.779" rpy="0 0 3.1416"/>
+    <origin xyz="1.027 0 0.779" rpy="0 0 3.1416"/> <!--z = 0.874 navigation -->
+    <!-- <origin xyz="... ... ..." rpy="0 0 3.1416"/> safety -->
   </joint>
   <!-- Revolute joint: base_link ↔ shaft (steering) -->
